File: electronics/Sumo/Sumo.kicad_pcb (KiCad board)
At the start: 2 copper layers, 60 x 100 mm, 8 parts, among them J1 EngineA, J2 EngineB, J3 QTR-8RC, J4 SHARP1, J5 SHARP2, U1 PololuMotorDriver

Commit message: Add files to control version
Routing:
- net VCC: track 133.3 -> 145.4 mm
Changed lines of the file:
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@@
   (general
     (links 39)
-    (no_connects 1)
+    (no_connects 0)
     (area 109.949999 74.949999 170.050001 175.050001)
     (thickness 1.6)
     (drawings 10)
-    (tracks 162)
+    (tracks 165)
     (zones 0)
     (modules 8)
@@
   (segment (start 119.46 111.76) (end 129.3914 101.8286) (width 0.5) (layer F.Cu) (net 3))
   (segment (start 129.3914 101.8286) (end 133.3411 101.8286) (width 0.5) (layer F.Cu) (net 3))
+  (segment (start 151.21 120.015) (end 151.21 122.762) (width 0.5) (layer B.Cu) (net 4) (status 400000))
+  (segment (start 152.273 123.825) (end 160.1 123.825) (width 0.5) (layer B.Cu) (net 4) (status 800000))
+  (segment (start 151.21 122.762) (end 152.273 123.825) (width 0.5) (layer B.Cu) (net 4))
   (segment (start 160.1 123.825) (end 163.91 123.825) (width 0.5) (layer F.Cu) (net 4))
   (segment (start 151.21 151.765) (end 151.21 156.21) (width 0.5) (layer F.Cu) (net 4))
@@
     (polygon
       (pts
-        (xy 162 81.365) (xy 167 81.365) (xy 168 166.365) (xy 162 166.365) (xy 162 172.365)
-        (xy 118 172.365) (xy 118 166.365) (xy 112 166.365) (xy 112.954023 85.273046) (xy 113 81.365)
-        (xy 115 81.365) (xy 118 81.365) (xy 118 76.365) (xy 162 76.365)
+        (xy 162.052 81.534) (xy 168.148 81.534) (xy 168.148 122.174) (xy 152.654 122.174) (xy 152.654 117.094)
+        (xy 149.606 117.094) (xy 149.606 126.492) (xy 168.148 126.492) (xy 168.148 167.64) (xy 161.798 167.64)
+        (xy 161.798 173.482) (xy 117.856 173.482) (xy 117.856 167.64) (xy 112.014 167.64) (xy 112.014 81.534)
+        (xy 118.364 81.534) (xy 118.364 76.708) (xy 162.052 76.708)
       )
     )

Commit message: Fix traces, add rounded edges, add mounting holes
Parts:
- added REF**: MountingHole_4mm, Mounting_Holes:MountingHole_4mm, F.Cu at (166.0, 171.0)
- added REF**: MountingHole_4mm, Mounting_Holes:MountingHole_4mm, F.Cu at (114.0, 171.0)
- added REF**: MountingHole_4mm, Mounting_Holes:MountingHole_4mm, F.Cu at (114.0, 78.0)
- added REF**: MountingHole_4mm, Mounting_Holes:MountingHole_4mm, F.Cu at (166.0, 78.0)
- added REF***: OSHW-Logo_5.7x6mm_SilkScreen, Symbols:OSHW-Logo_5.7x6mm_SilkScreen, F.Cu at (122.5, 171.1)
Routing:
- net Net-(SH1-Pad10): track 36.1 -> 34.2 mm
- net BIN1: track 37.0 -> 35.2 mm
- net Net-(SH1-Pad11): track 65.6 -> 66.9 mm
- net Net-(J3-Pad3): track 28.0 -> 26.7 mm
- net BIN2: track 34.8 -> 33.7 mm
- added copper zone on F.Cu, net VCC
Other:
- outline, holes or cut-outs redrawn

Commit message: Add logo to PCB
Parts:
- added G***: LOGO, Sumo:logo, B.Cu at (138.6, 122.3)
